Commit message: added function to plot multiple sets of base_parameters at once

File: URe/urdf/ur10e.urdf (robot description, URDF)
Before this commit: robot ur10e, 11 links, 10 joints
Links:
- link base_link: geometry collision mesh filename=../meshes/ur10e/collision/base.stl; visual mesh filename=../meshes/ur10e/visual/base.dae
- link forearm_link: geometry collision mesh filename=../meshes/ur10e/collision/forearm.stl; visual mesh filename=../meshes/ur10e/visual/forearm.dae
- link shoulder_link: geometry collision mesh filename=../meshes/ur10e/collision/shoulder.stl; visual mesh filename=../meshes/ur10e/visual/shoulder.dae
- link upper_arm_link: geometry collision mesh filename=../meshes/ur10e/collision/upperarm.stl; visual mesh filename=../meshes/ur10e/visual/upperarm.dae
- link wrist_1_link: geometry collision mesh filename=../meshes/ur10e/collision/wrist1.stl; visual mesh filename=../meshes/ur10e/visual/wrist1.dae
- link wrist_2_link: geometry collision mesh filename=../meshes/ur10e/collision/wrist2.stl; visual mesh filename=../meshes/ur10e/visual/wrist2.dae
- link wrist_3_link: geometry collision mesh filename=../meshes/ur10e/collision/wrist3.stl; visual mesh filename=../meshes/ur10e/visual/wrist3.dae
