Commit message: n dof

File: urdf/fixed_bipedal.urdf (robot description, URDF)
Before this commit: robot fixed_bipedal, 13 links, 12 joints
Joints:
- joint L_Hip_Pitch: axis 0. 1. 0. -> 0 1 0
- joint L_Hip_Roll: axis 1. 0. 0. -> 1 0 0
- joint L_Hip_Yaw: axis 0. 0. 1. -> 0 0 1
- joint L_Knee_Pitch: axis 0. 1. 0. -> 0 1 0
- joint R_Hip_Pitch: axis 0. 1. 0. -> 0 1 0
- joint R_Hip_Roll: axis 1. 0. 0. -> 1 0 0
- joint R_Hip_Yaw: axis 0. 0. 1. -> 0 0 1
- joint R_Knee_Pitch: axis 0. 1. 0. -> 0 1 0
